File: hrsens/hrsens.kicad_pcb (KiCad board)
At the start: 2 copper layers, 69.8 x 97.9 mm, 5 parts, among them U1 ENS160-BGLM, U2 XIAO-RP2040-DIP, U3 OLED_0.91_128x32

Commit message: ok bye guys! pcb out
- silkscreened some stuffs
- touched up some traces again
tapping out for tonight bluds. i forgot about my homework that was definitely due tomorrow so
Parts:
- added G***: LOGO, LOGO, F.Cu at (74.5, 93.2)
- added G***: LOGO, LOGO, F.Cu at (73.5, 99.6)
- added G***: LOGO, LOGO, F.Cu at (77.9, 86.9)
- added G***: LOGO, LOGO, B.Cu at (109.5, 64.0)
Other:
- board text added: "made with <3 by sua for hermes"
