File: aqkitty!/hrsens.kicad_pcb (KiCad board)
At the start: 2 copper layers, 69.8 x 97.9 mm, 9 parts, among them U1 ENS160-BGLM, U2 XIAO-RP2040-DIP, U3 OLED_0.91_128x32

Commit message: final touches?
added a mounting hole because why not, i think im done
Parts:
- added REF**: MountingHole_3mm, MountingHole:MountingHole_3mm, F.Cu at (109.5, 47.5)

Commit message: fix.. and layout...
added pullups, temp sensor, then started the NIGHTMARE that is pcb layout
Parts:
- added C1: 10uF, Capacitor_SMD:C_0603_1608Metric_Pad1.08x0.95mm_HandSolder, F.Cu at (150.7, 90.8)
- added C2: 10uF, Capacitor_SMD:C_0603_1608Metric_Pad1.08x0.95mm_HandSolder, F.Cu at (150.7, 93.3)
- added C3: 0.1uF, Capacitor_SMD:C_0603_1608Metric_Pad1.08x0.95mm_HandSolder, F.Cu at (150.7, 95.8)
- added D1: LED, LED_SMD:LED_0603_1608Metric_Pad1.05x0.95mm_HandSolder, F.Cu at (155.1, 94.8)
- added R3: R, Resistor_SMD:R_0603_1608Metric_Pad0.98x0.95mm_HandSolder, F.Cu at (150.7, 98.3)
- added U4: SHT30-DIS, Sensor_Humidity:Sensirion_DFN-8-1EP_2.5x2.5mm_P0.5mm_EP1.1x1.7mm, F.Cu at (155.3, 91.5)
Connections:
- net /3V3 renamed +3V3
- net VSS renamed GND
- U2 pad 1: unconnected-(U2-GPIO26/ADC0/A0-Pad1)_1 -> Net-(U2-GPIO26/ADC0/A0)
Routing:
- net +3V3: track 77.1 -> 0.00 mm
- net /SCL: track 69.6 -> 0.00 mm
- net /SDA: track 65.8 -> 0.00 mm
- net GND: track 48.3 -> 0.00 mm, vias 2 -> 0
