File: aqkitty!/hrsens.kicad_pcb (KiCad board)
At the start: 2 copper layers, 69.8 x 97.9 mm, 16 parts, among them U1 ENS160-BGLM, U2 XIAO-RP2040-DIP, U3 OLED_0.91_128x32, U4 SHT30-DIS

Commit message: yay finished pcb layout
for REAL this time after adding temp sens and also um yes gonna do readme now
Parts:
- R3: value R -> 330R
- U1: value ENS160-BGLM -> ENS160
- U4: value SHT30-DIS -> SHT30
- moved U1 47.8 mm to (84.8, 126.9), turned to 0 degrees
- moved U4 46.7 mm to (84.5, 120.5)
- moved C2 37.3 mm to (90.2, 125.9), turned to 0 degrees
- moved C3 35.6 mm to (91.5, 121.2), turned to 0 degrees
- moved R1 17.1 mm to (91.0, 115.3)
- moved R2 15.5 mm to (92.0, 131.6)
- moved C1 9.59 mm to (85.6, 131.5), turned to 0 degrees
- moved D1 7.32 mm to (127.1, 131.8)
- moved U2 7.17 mm to (114.5, 124.3)
- moved R3 5.25 mm to (127.2, 127.6), turned to 180 degrees
- moved U3 1.35 mm to (91.3, 102.9)
Connections:
- net /SCL renamed SCL
- net /SDA renamed SDA
- D1 pad 1: Net-(D1-A) -> Net-(D1-K)
- R3 pad 2: Net-(D1-A) -> Net-(D1-K)
- U4 pad 6: GND -> +3V3
Routing:
- net GND: track 77.6 -> 12.6 mm, vias 13 -> 4
- net SDA: track 127.6 -> 111.7 mm
- net +3V3: track 115.0 -> 103.8 mm, vias 1 -> 3
- net Net-(D1-A): track 15.9 -> 5.94 mm, vias 1 -> 0
- net SCL: track 103.5 -> 98.6 mm, vias 2 -> 1
- net Net-(D1-K): track 0.00 -> 4.22 mm
