File: aqkitty!/hrsens.kicad_sch (KiCad schematic)
At the start: 5 parts, among them U1 ENS160-BGLM, U2 XIAO-RP2040-DIP, U3 OLED_0.91_128x32

Commit message: fix.. and layout...
added pullups, temp sensor, then started the NIGHTMARE that is pcb layout
Parts:
- added C1, C2: 10uF, Capacitor_SMD:C_0603_1608Metric_Pad1.08x0.95mm_HandSolder, symbol Device:C
- added C3: 0.1uF, Capacitor_SMD:C_0603_1608Metric_Pad1.08x0.95mm_HandSolder, symbol Device:C
- added D1: LED, LED_SMD:LED_0603_1608Metric_Pad1.05x0.95mm_HandSolder, symbol Device:LED
- added R3: R, Resistor_SMD:R_0603_1608Metric_Pad0.98x0.95mm_HandSolder, symbol Device:R
- added U4: SHT30-DIS, Sensor_Humidity:Sensirion_DFN-8-1EP_2.5x2.5mm_P0.5mm_EP1.1x1.7mm, symbol Sensor_Humidity:SHT30-DIS
Connections:
- net SCL: now also U4.4 (SCL)
- net SDA: now also U4.1 (SDA)
- net at U2.1 (GPIO26/ADC0/A0): now also R3.2
- net 3V3 renamed +3V3
- net +3V3: now also C1.1, C2.1, C3.1, U4.2 (ADDR), U4.5 (VDD)
- net VSS renamed GND
- net GND: now also C1.2, C2.2, C3.2, D1.1 (K), U4.6 (~{RESET}), U4.8 (VSS), U4.9 (VSS)
- new net: D1.2 (A), R3.1
- no-connect marks 11 -> 10
Other:
- moved on the sheet: R2, U1
